File: pcb/doorbell.kicad_pcb (KiCad board)
At the start: 2 copper layers, 44.9 x 59.2 mm, 12 parts, among them J1 USB-C Breakout Board, SW1 SW_Push, U1 ESP32-CAM, U2 MAX9814

Commit message: added my silkscreen art!!
Parts:
- added G***: LOGO, logo:hc, F.Cu at (121.0, 89.0)
Other:
- board text added: "POWERED BY"
- board text added: "SECURODOOR"
